Commit message: Added meshes and urdf

File: auto_quad_description/urdf/auto_quad.urdf (robot description, URDF)
Before this commit: robot auto_quad, 5 links, 4 joints
Links:
- added link back_left_propeller; collision cylinder length=0.005 radius=0.05; visual mesh filename=package://auto_quad_description/meshes/propeller.stl scale=0.01 0.01 0.01
- added link back_right_propeller; collision cylinder length=0.005 radius=0.05; visual mesh filename=package://auto_quad_description/meshes/propeller.stl scale=0.01 0.01 0.01
- added link front_left_propeller; collision cylinder length=0.005 radius=0.05; visual mesh filename=package://auto_quad_description/meshes/propeller.stl scale=0.01 0.01 0.01
- added link front_right_propeller; collision cylinder length=0.005 radius=0.05; visual mesh filename=package://auto_quad_description/meshes/propeller.stl scale=0.01 0.01 0.01
- added link lidar_link; collision mesh filename=package://auto_quad_description/meshes/laser_link.stl scale=0.01 0.01 0.01; visual mesh filename=package://auto_quad_description/meshes/laser_link.stl scale=0.01 0.01 0.01
- added link pi_case; collision mesh filename=package://auto_quad_description/meshes/pi_case.stl scale=0.01 0.01 0.01; visual mesh filename=package://auto_quad_description/meshes/pi_case.stl scale=0.01 0.01 0.01
- added link world
- link back_left_motor: mass 0.1 -> None; geometry collision cylinder length=0.02 radius=0.01; visual mesh filename=package://auto_quad_description/meshes/motor.stl scale=0.01 0.01 0.01
- link back_right_motor: mass 0.1 -> None; geometry collision cylinder length=0.02 radius=0.01; visual mesh filename=package://auto_quad_description/meshes/motor.stl scale=0.01 0.01 0.01
- link base_link: mass 1.0 -> None; geometry collision mesh filename=package://auto_quad_description/meshes/quadcopter_frame.stl scale=0.01 0.01 0.01; visual mesh filename=package://auto_quad_description/meshes/quadcopter_frame.stl scale=0.01 0.01 0.01
- link front_left_motor: mass 0.1 -> None; geometry collision cylinder length=0.02 radius=0.01; visual mesh filename=package://auto_quad_description/meshes/motor.stl scale=0.01 0.01 0.01
- link front_right_motor: mass 0.1 -> None; geometry collision cylinder length=0.02 radius=0.01; visual mesh filename=package://auto_quad_description/meshes/motor.stl scale=0.01 0.01 0.01
Joints:
- added joint back_left_propeller_joint: type continuous, parent back_left_motor, child back_left_propeller, origin xyz=0 0 0 rpy=0 0 0, axis 0 0 1
- added joint back_right_propeller_joint: type continuous, parent back_right_motor, child back_right_propeller, origin xyz=0 0 0 rpy=0 0 0, axis 0 0 1
- added joint base_to_world: type fixed, parent world, child base_link, origin xyz=0 0 0 rpy=0 0 0
- added joint front_left_propeller_joint: type continuous, parent front_left_motor, child front_left_propeller, origin xyz=0 0 0 rpy=0 0 0, axis 0 0 1
- added joint front_right_propeller_joint: type continuous, parent front_right_motor, child front_right_propeller, origin xyz=0 0 0 rpy=0 0 0, axis 0 0 1
- added joint lidar_joint: type fixed, parent base_link, child lidar_link, origin xyz=-0.2 0 0.53 rpy=0 0 0
- added joint pi_case_joint: type fixed, parent base_link, child pi_case, origin xyz=0 0 0 rpy=0 0 0
- joint back_left_motor_joint: origin xyz=0.1 -0.1 0 rpy=0 0 0 -> xyz=-1.58 1.58 0.18 rpy=0 0 0
- joint back_right_motor_joint: origin xyz=-0.1 -0.1 0 rpy=0 0 0 -> xyz=-1.58 -1.58 0.18 rpy=0 0 0
- joint front_left_motor_joint: origin xyz=0.1 0.1 0 rpy=0 0 0 -> xyz=1.58 1.58 0.18 rpy=0 0 0
- joint front_right_motor_joint: origin xyz=-0.1 0.1 0 rpy=0 0 0 -> xyz=1.58 -1.58 0.18 rpy=0 0 0

Commit message: Added localization

File: auto_quad_description/urdf/auto_quad.urdf (robot description, URDF)
Before this commit: robot auto_quad, 12 links, 11 joints
Links:
- added link stereo_camera_link; collision mesh filename=package://auto_quad_description/meshes/3d_stereo_camera.stl scale=0.01 0.01 0.01; visual mesh filename=package://auto_quad_description/meshes/3d_stereo_camera.stl scale=0.01 0.01 0.01
Joints:
- added joint stereo_camera_joint: type fixed, parent base_link, child stereo_camera_link, origin xyz=0.35 0 0.25 rpy=1.5708 0 1.5708
